File: mini-dvhstx.kicad_pcb (KiCad board)
At the start: 4 copper layers, 20.6 x 49.4 mm, 46 parts, among them J1 USB-C, J2 HDMI_A, J3 Conn_01x15, J5 Conn_01x15, U1 RP2350_60QFN, U2 AP2112K-3.3, U3 W25Q32JV, Y1 ABM8-272-T3

Commit message: Redesign
Parts:
- BTN1: renamed from BOOT; value SW_Push -> BOOT
- BTN2: renamed from RESET; value SW_Push -> RESET
- J3: value Conn_01x15 -> Conn_01x16
- J5: value Conn_01x15 -> Conn_01x13
- moved R9 11.6 mm to (80.6, 125.6), turned to 180 degrees
- moved D1 9.23 mm to (82.5, 124.5)
- moved J2 4.67 mm to (86.6, 136.1)
- moved R12 4.19 mm to (84.7, 129.2)
- moved R13 4.19 mm to (85.8, 129.2)
- moved R14 4.19 mm to (86.8, 129.2)
- moved R15 4.19 mm to (87.8, 129.2)
- moved R17 4.19 mm to (89.8, 129.2)
- moved R18 4.19 mm to (90.8, 129.2)
- moved R16 4.19 mm to (88.8, 129.2)
- moved R19 4.19 mm to (91.9, 129.2)
- moved C18 0.38 mm to (86.4, 126.0)
- moved C16 0.36 mm to (90.6, 124.6)
- moved C10 0.34 mm to (87.4, 126.0)
Connections:
- J2 pad 19: unconnected-(J2-HPD-Pad19) -> /HDMI_HPD
- J3 pad 11: /GPIO9 -> /GPIO8
- J3 pad 12: /GPIO8 -> /GPIO9
- J5 pad 10: /GPIO26_ADC0 -> /GPIO22
- J5 pad 11: /GPIO23 -> /SWD
- J5 pad 12: /GPIO22 -> /SWCLK
- J5 pad 9: /GPIO27_ADC1 -> /GPIO23
Routing:
- net /SWCLK: track 0.00 -> 8.97 mm, vias 0 -> 1
- net /SWD: track 0.00 -> 8.51 mm, vias 0 -> 1
- net /GPIO19: track 0.00 -> 6.61 mm
- net /GPIO15: track 0.00 -> 6.61 mm
- net /GPIO14: track 0.00 -> 6.24 mm
- net /GPIO18: track 0.00 -> 5.98 mm
- net /GPIO13: track 0.00 -> 5.95 mm
- net /GPIO16: track 0.00 -> 5.86 mm
- net /GPIO17: track 0.00 -> 5.73 mm
- net /GPIO12: track 0.00 -> 5.66 mm
- net Net-(J2-CK-): track 0.00 -> 3.40 mm
- net Net-(J2-CK+): track 0.00 -> 3.40 mm
- net Net-(J2-D2+): track 0.00 -> 3.38 mm
- net Net-(J2-D2-): track 0.00 -> 3.38 mm
- net Net-(J2-D0-): track 0.00 -> 3.18 mm
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- added copper zone on F.Cu, net +3V3
Other:
- board size 20.6 x 49.4 mm -> 20.6 x 44.2 mm

Commit message: Complete routing
Parts:
- BTN2: value RESET -> RST
- moved R4 1.86 mm to (81.3, 115.2), turned to 90 degrees
- moved C1 1.32 mm to (88.1, 107.4)
- moved R9 1.10 mm to (80.2, 124.6)
- moved C13 0.72 mm to (83.1, 115.1)
- moved C8 0.40 mm to (82.5, 118.9), turned to 180 degrees
- moved C15 0.36 mm to (82.5, 120.9), turned to 180 degrees
- moved C10 0.36 mm to (87.5, 126.3)
- moved C4 0.18 mm to (82.4, 129.8)
- moved BTN2 0.15 mm to (79.9, 119.7)
- moved D1 0.15 mm to (82.7, 124.6), turned to 0 degrees
- moved C3 0.10 mm to (82.4, 127.0)
- moved C11 0.10 mm to (91.9, 118.8)
- moved C14 0.10 mm to (91.9, 120.3)
- moved R3 0.05 mm to (83.4, 129.0)
Routing:
- net /HDMI_5V: track 0.00 -> 52.2 mm, vias 0 -> 1
- net /GPIO0: track 0.00 -> 22.0 mm, vias 0 -> 1
- net +3V3: track 5.06 -> 25.6 mm, vias 0 -> 9
- net /GPIO1: track 0.00 -> 20.3 mm, vias 0 -> 1
- net /GPIO11: track 0.00 -> 16.6 mm, vias 0 -> 1
- net /GPIO2: track 0.00 -> 15.8 mm, vias 0 -> 1
- net GND: track 14.5 -> 29.9 mm, vias 10 -> 23
- net /GPIO10: track 0.00 -> 14.6 mm, vias 0 -> 1
- net /GPIO3: track 0.00 -> 13.8 mm, vias 0 -> 1
- net /GPIO4: track 0.00 -> 12.6 mm
- net GPIO20: track 0.00 -> 11.2 mm, vias 0 -> 2
- net /GPIO9: track 0.00 -> 11.2 mm
- net /GPIO5: track 0.00 -> 10.5 mm
- net /RUN: track 1.39 -> 11.1 mm, vias 1 -> 2
- net /GPIO8: track 0.00 -> 9.10 mm
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- added copper zone on B.Cu, net +1V1
- added copper zone on In2.Cu, net +3V3
- added copper zone on F.Cu, net +5V
- added copper zone on B.Cu, net GND
- added copper zone on F.Cu, net GND
- added copper zone on In1.Cu, net GND
- added copper zone on In2.Cu, net GND

Commit message: Silkscreen
Connections:
- J2 pad 20: (no net) -> GND
- J2 pad 21: (no net) -> GND
- J2 pad 22: (no net) -> GND
- J2 pad 23: (no net) -> GND
Other:
- board text added: "0"
- board text added: "1"
- board text added: "10"
- board text added: "11"
- board text added: "2"
- board text added: "22"
- board text added: "23"
- board text added: "28"
- board text added: "29"
- board text added: "3"
- board text added: "3V3"
- board text added: "4"
- board text added: "5"
- board text added: "6"
- board text added: "7"
- board text added: "8"
- board text added: "9"
- board text added: "GND"
- board text added: "HDMI 5V"
- board text added: "HDMI HPD"
- board text added: "JLCJLCJLCJLC"
- board text added: "Mini DV HSTX"
- board text added: "Not HDMI just sparkling DVI"
- board text added: "SWC"
- board text added: "SWD"
- board text added: "VBUS"
- board text added: "design by RebelMike"
