File: mini-dvhstx.kicad_pcb (KiCad board)
At the start: 4 copper layers, 20.6 x 44.2 mm, 46 parts, among them J1 USB-C, J2 HDMI_A, J3 Conn_01x16, J5 Conn_01x13, U1 RP2350_60QFN, U2 AP2112K-3.3, U3 W25Q32JV, Y1 ABM8-272-T3

Commit message: Tweaks
Parts:
- added C2: 100n, Capacitor_SMD:C_0201_0603Metric, F.Cu at (84.3, 108.2)
- moved C5 7.87 mm to (92.0, 109.0), turned to 90 degrees
- moved C1 1.73 mm to (89.2, 106.0), turned to 180 degrees
- moved U2 0.54 mm to (89.8, 108.5)
Routing:
- net +3V3: track 25.6 -> 28.0 mm
- net +5V: track 14.0 -> 12.4 mm
- net Net-(J1-CC1): track 8.71 -> 9.54 mm
- net GND: track 29.9 -> 29.8 mm, vias 23 -> 24

Commit message: Moving towards v1
Parts:
- added TP1: TestPoint, TestPoint:TestPoint_Pad_2.0x2.0mm, B.Cu at (88.3, 111.5)
- C3, C4: value 15p -> 13p
- moved R19 1.95 mm to (91.4, 127.3)
Routing:
- net /GPIO19: track 6.61 -> 4.54 mm
- net Net-(J2-D2+): track 3.38 -> 5.11 mm

Commit message: First version
Other:
- board size 20.6 x 44.2 mm -> 20.8 x 47.4 mm
- board text added: "1V1"
Changed lines of the file:
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@@
 			(at 0 1.998 0)
 			(layer "B.SilkS")
+			(hide yes)
 			(effects
 				(font
@@
 	)
 	(gr_line
-		(start 94.107 141.605)
-		(end 76.073 141.605)
+		(start 94.107 144.399)
+		(end 75.819 144.399)
 		(stroke
 			(width 0.05)
@@
 	)
 	(gr_line
-		(start 74.803 140.335)
-		(end 74.803 98.425)
+		(start 74.549 143.129)
+		(end 74.549 98.044)
 		(stroke
 			(width 0.05)
@@
 	)
 	(gr_arc
-		(start 95.377 140.335)
-		(mid 95.005026 141.233026)
-		(end 94.107 141.605)
+		(start 95.377 143.129)
+		(mid 95.005026 144.027026)
+		(end 94.107 144.399)
 		(stroke
 			(width 0.05)
@@
 	)
 	(gr_arc
-		(start 76.073 141.605)
-		(mid 75.174974 141.233026)
-		(end 74.803 140.335)
+		(start 75.819 144.399)
+		(mid 74.920974 144.027026)
+		(end 74.549 143.129)
 		(stroke
 			(width 0.05)
@@
 	)
 	(gr_arc
-		(start 94.361 97.409)
-		(mid 95.07942 97.70658)
-		(end 95.377 98.425)
+		(start 94.361 97.028)
+		(mid 95.07942 97.32558)
+		(end 95.377 98.044)
 		(stroke
 			(width 0.05)
@@
 	)
 	(gr_line
-		(start 95.377 98.425)
-		(end 95.377 140.335)
+		(start 95.377 98.044)
+		(end 95.377 143.129)
 		(stroke
 			(width 0.05)
@@
 	)
 	(gr_arc
-		(start 74.803 98.425)
-		(mid 75.10058 97.70658)
-		(end 75.819 97.409)
+		(start 74.549 98.044)
+		(mid 74.84658 97.32558)
+		(end 75.565 97.028)
 		(stroke
 			(width 0.05)
@@
 	)
 	(gr_line
-		(start 75.819 97.409)
-		(end 94.361 97.409)
+		(start 75.565 97.028)
+		(end 94.361 97.028)
 		(stroke
 			(width 0.05)
@@
 		)
 	)
+	(gr_text "1V1"
+		(at 89.6 110.2 0)
+		(layer "B.SilkS")
+		(effects
+			(font
+				(size 1 1)
+				(thickness 0.1)
+			)
+			(justify left bottom mirror)
+		)
+	)
 	(gr_text "10"
 		(at 82.296 132.715 0)
@@
 		(polygon
 			(pts
-				(xy 84.455 96.52) (xy 84.455 103.4288) (xy 96.52 103.4034) (xy 96.52 96.52)
+				(xy 84.455 97.5868) (xy 84.455 103.4288) (xy 96.52 103.4034) (xy 96.52 97.5868)
 			)
 		)
@@
 		(polygon
 			(pts
-				(xy 73.66 96.52) (xy 91.948 96.52) (xy 91.948 103.251) (xy 96.52 103.2764) (xy 96.52 142.24) (xy 73.66 142.24)
+				(xy 73.6092 97.5868) (xy 91.8972 97.5868) (xy 91.948 103.251) (xy 96.52 103.2764) (xy 96.52 142.24)
+				(xy 73.66 142.24)
 			)
 		)
