File: mini-dvhstx.kicad_sch (KiCad schematic)
At the start: 46 parts, among them J1 USB-C, J2 HDMI_A, J3 Conn_01x15, J5 Conn_01x15, SW1 SW_Push, U1 RP2350_60QFN, U2 AP2112K-3.3, U3 W25Q32JV, Y1 ABM8-272-T3

Commit message: Redesign
Parts:
- removed J5: Conn_01x15, Connector_PinHeader_2.54mm:PinHeader_1x15_P2.54mm_Vertical, symbol Connector_Generic:Conn_01x15
- added J5: Conn_01x13, Connector_PinHeader_2.54mm:PinHeader_1x15_P2.54mm_Vertical, symbol Connector_Generic:Conn_01x13
- BTN2: renamed from RST1; value SW_Push -> RESET
- J3: value Conn_01x15 -> Conn_01x16; symbol Connector_Generic:Conn_01x15 -> Connector_Generic:Conn_01x16
- SW1: value SW_Push -> BOOT
Connections:
- net +3V3: now also J5.5 (Pin_5)
- net +5V: now also J5.1 (Pin_1)
- net GND: now also J5.13 (Pin_13), J5.3 (Pin_3), J5.8 (Pin_8)
- net GPIO22: now also J5.10 (Pin_10)
- net GPIO23: now also J5.9 (Pin_9)
- net GPIO28_ADC2: now also J5.7 (Pin_7)
- net GPIO29_ADC3: now also J5.6 (Pin_6)
- net GPIO8: now also J3.11 (Pin_11); no longer J3.12 (Pin_12)
- net GPIO9: now also J3.12 (Pin_12); no longer J3.11 (Pin_11)
- net HDMI_5V: now also J5.2 (Pin_2)
- net SWCLK: now also J5.12 (Pin_12)
- net SWD: now also J5.11 (Pin_11)
- net HDMI_HPD: now reaches J2.19 (HPD)
- net HDMI_HPD: now also J3.16 (Pin_16)
- no-connect marks 11 -> 10

Commit message: Complete routing
Parts:
- BTN2: value RESET -> RST
Changed lines of the file:
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@@
 			)
 		)
-		(property "Value" "RESET"
+		(property "Value" "RST"
 			(at 144.78 160.02 0)
 			(effects

Commit message: Add schematic
Other:
- company: (none) -> Team Rebellion
- title: (none) -> Mini DV HSTX
Changed lines of the file:
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@@
 	(generator_version "8.0")
 	(paper "A3")
+	(title_block
+		(title "Mini DV HSTX")
+		(date "2025-02-15")
+		(rev "v1.0")
+		(company "Team Rebellion")
+	)
 	(junction
 		(at 152.4 252.73)

Commit message: Tweaks
Parts:
- added C2: 100n, Capacitor_SMD:C_0201_0603Metric, symbol Device:C
- U3: JLC C97521 -> C571260
Connections:
- net +3V3: now also C2.1
- net GND: now also J2.20 (SH), J2.21 (SH), J2.22 (SH), J2.23 (SH), C2.2; no longer J2.SH
Changed lines of the file:
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@@
 	)
 	(junction
+		(at 73.66 107.95)
+		(diameter 0)
+		(color 0 0 0 0)
+	)
+	(junction
 		(at 152.4 260.35)
 		(diameter 0)
@@
 	(wire
 		(pts
+			(xy 73.66 107.95) (xy 73.66 123.19)
+		)
+		(stroke
+			(width 0)
+			(type default)
+		)
+	)
+	(wire
+		(pts
 			(xy 325.12 118.11) (xy 325.12 129.54)
 		)
@@
 	(wire
 		(pts
-			(xy 73.66 105.41) (xy 73.66 123.19)
+			(xy 73.66 105.41) (xy 73.66 107.95)
 		)
 		(stroke
@@
 	(wire
 		(pts
+			(xy 87.63 107.95) (xy 73.66 107.95)
+		)
+		(stroke
+			(width 0)
+			(type default)
+		)
+	)
+	(wire
+		(pts
 			(xy 337.82 119.38) (xy 332.74 119.38)
 		)
@@
 	(wire
 		(pts
+			(xy 87.63 119.38) (xy 87.63 123.19)
+		)
+		(stroke
+			(width 0)
+			(type default)
+		)
+	)
+	(wire
+		(pts
 			(xy 213.36 252.73) (xy 222.25 252.73)
 		)
@@
 	(wire
 		(pts
+			(xy 87.63 111.76) (xy 87.63 107.95)
+		)
+		(stroke
+			(width 0)
+			(type default)
+		)
+	)
+	(wire
+		(pts
 			(xy 205.74 233.68) (xy 205.74 242.57)
 		)
@@
 			)
 		)
-		(property "JLC" "C97521"
+		(property "JLC" "C571260"
 			(at 73.66 135.89 0)
 			(effects
@@
 	(symbol
 		(lib_id "power:GND")
+		(at 87.63 123.19 0)
+		(mirror y)
+		(unit 1)
+		(exclude_from_sim no)
+		(in_bom yes)
+		(on_board yes)
+		(dnp no)
+		(property "Reference" "#PWR010"
+			(at 87.63 129.54 0)
+			(effects
+				(font
+					(size 1.27 1.27)
+				)
+				(hide yes)
+			)
+		)
+		(property "Value" "GND"
+			(at 91.44 124.46 0)
+			(effects
+				(font
+					(size 1.27 1.27)
+				)
+			)
+		)
+		(property "Footprint" ""
+			(at 87.63 123.19 0)
+			(effects
+				(font
+					(size 1.27 1.27)
+				)
+				(hide yes)
+			)
+		)
+		(property "Datasheet" ""
+			(at 87.63 123.19 0)
+			(effects
+				(font
+					(size 1.27 1.27)
+				)
+				(hide yes)
+			)
+		)
+		(property "Description" ""
+			(at 87.63 123.19 0)
+			(effects
+				(font
+					(size 1.27 1.27)
+				)
+				(hide yes)
+			)
+		)
+		(pin "1"
+		)
+		(instances
+			(project "mini-dvhstx"
+				(path "/ead8f88d-5617-4ec7-a65f-e9d77c3564d6"
+					(reference "#PWR010")
+					(unit 1)
+				)
+			)
+		)
+	)
+	(symbol
+		(lib_id "power:GND")
 		(at 43.18 76.2 0)
 		(unit 1)
@@
 		(pin "3"
 		)
-		(pin "SH"
+		(pin "20"
 		)
 		(pin "1"
@@
 		(pin "8"
 		)
+		(pin "23"
+		)
+		(pin "21"
+		)
+		(pin "22"
+		)
 		(instances
 			(project ""
@@
 					(unit 1)
 				)
+			)
+		)
+	)
+	(symbol
+		(lib_id "Device:C")
+		(at 87.63 115.57 0)
+		(unit 1)
+		(exclude_from_sim no)
+		(in_bom yes)
+		(on_board yes)
+		(dnp no)
+		(property "Reference" "C2"
+			(at 90.551 114.4016 0)
+			(effects
+				(font
+					(size 1.27 1.27)
+				)
+				(justify left)
+			)
+		)
+		(property "Value" "100n"
+			(at 90.551 116.713 0)
+			(effects
+				(font
+					(size 1.27 1.27)
+				)
+				(justify left)
+			)
+		)
+		(property "Footprint" "Capacitor_SMD:C_0201_0603Metric"
+			(at 88.5952 119.38 0)
+			(effects
+				(font
+					(size 1.27 1.27)
+				)
+				(hide yes)
+			)
+		)
+		(property "Datasheet" "~"
+			(at 87.63 115.57 0)
+			(effects
+				(font
+					(size 1.27 1.27)
+				)
+				(hide yes)
+			)
+		)
+		(property "Description" ""
+			(at 87.63 115.57 0)
+			(effects
+				(font
+					(size 1.27 1.27)
+				)
+				(hide yes)
+			)
+		)
+		(pin "1"
+		)
+		(pin "2"
+		)
+		(instances
+			(project "mini-dvhstx"
+				(path "/ead8f88d-5617-4ec7-a65f-e9d77c3564d6"
+					(reference "C2")
+					(unit 1)
+				)

Commit message: Moving towards v1
Parts:
- added TP1: TestPoint, TestPoint:TestPoint_Pad_2.0x2.0mm, symbol Connector:TestPoint
- C3, C4: value 15p -> 13p; JLC (none) -> C48936
- U1: JLC (none) -> C42411118
Connections:
- net +1V1: now also TP1.1
Changed lines of the file:
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@@
 	)
 	(junction
+		(at 143.51 60.96)
+		(diameter 0)
+		(color 0 0 0 0)
+	)
+	(junction
 		(at 196.85 81.28)
 		(diameter 0)
@@
 	(wire
 		(pts
+			(xy 130.81 60.96) (xy 143.51 60.96)
+		)
+		(stroke
+			(width 0)
+			(type default)
+		)
+	)
+	(wire
+		(pts
 			(xy 69.215 229.87) (xy 66.675 229.87)
 		)
@@
 			)
 		)
-		(property "Description" ""
+		(property "Description" "RP2350A"
+			(at 198.12 144.78 0)
+			(effects
+				(font
+					(size 1.27 1.27)
+				)
+				(hide yes)
+			)
+		)
+		(property "JLC" "C42411118"
 			(at 198.12 144.78 0)
 			(effects
@@
 			)
 		)
-		(property "Value" "15p"
+		(property "Value" "13p"
 			(at 71.882 242.951 0)
 			(effects
@@
 			)
 		)
+		(property "JLC" "C48936"
+			(at 73.025 240.03 0)
+			(effects
+				(font
+					(size 1.27 1.27)
+				)
+				(hide yes)
+			)
+		)
 		(pin "1"
 		)
@@
 	)
 	(symbol
+		(lib_id "Connector:TestPoint")
+		(at 130.81 60.96 0)
+		(unit 1)
+		(exclude_from_sim no)
+		(in_bom yes)
+		(on_board yes)
+		(dnp no)
+		(fields_autoplaced yes)
+		(property "Reference" "TP1"
+			(at 133.35 56.3879 0)
+			(effects
+				(font
+					(size 1.27 1.27)
+				)
+				(justify left)
+			)
+		)
+		(property "Value" "TestPoint"
+			(at 133.35 58.9279 0)
+			(effects
+				(font
+					(size 1.27 1.27)
+				)
+				(justify left)
+			)
+		)
+		(property "Footprint" "TestPoint:TestPoint_Pad_2.0x2.0mm"
+			(at 135.89 60.96 0)
+			(effects
+				(font
+					(size 1.27 1.27)
+				)
+				(hide yes)
+			)
+		)
+		(property "Datasheet" "~"
+			(at 135.89 60.96 0)
+			(effects
+				(font
+					(size 1.27 1.27)
+				)
+				(hide yes)
+			)
+		)
+		(property "Description" "test point"
+			(at 130.81 60.96 0)
+			(effects
+				(font
+					(size 1.27 1.27)
+				)
+				(hide yes)
+			)
+		)
+		(pin "1"
+		)
+		(instances
+			(project ""
+				(path "/ead8f88d-5617-4ec7-a65f-e9d77c3564d6"
+					(reference "TP1")
+					(unit 1)
+				)
+			)
+		)
+	)
+	(symbol
 		(lib_id "power:VBUS")
 		(at 332.74 118.11 0)
@@
 			)
 		)
-		(property "Value" "15p"
+		(property "Value" "13p"
 			(at 71.882 232.791 0)
 			(effects
@@
 			(at 73.025 229.87 0)
 			(effects
+				(font
+					(size 1.27 1.27)
+				)
+				(hide yes)
+			)
+		)
+		(property "JLC" "C48936"
+			(at 73.025 229.87 0)
+			(effects
