File: ram-pack.kicad_pcb (KiCad board)
At the start: 4 copper layers, 20.6 x 41.7 mm, 12 parts, among them J1 Conn_01x09, J2 Conn_01x15, J3 DEBUG, J4 QwST, U1 878-APS6404L-3SQR-SN, U2 878-APS6404L-3SQR-SN

Commit message: Moving towards v1
Parts:
- J4: footprint Connector_JST:JST_SH_SM04B-SRSS-TB_1x04-1MP_P1.00mm_Horizontal -> Connector_JST:JST_SH_BM04B-SRSS-TB_1x04-1MP_P1.00mm_Vertical
- moved J4 0.34 mm to (84.9, 59.3), turned to 0 degrees
Routing:
- net /SDA: track 22.6 -> 27.8 mm
- net +3V3: track 5.13 -> 9.14 mm, vias 1 -> 4
- net /SCL: track 19.5 -> 21.7 mm
- added copper zone on In2.Cu, net +3V3
Other:
- outline, holes or cut-outs redrawn
