File: ram-pack.kicad_sch (KiCad schematic)
At the start: 12 parts, among them J1 Conn_01x09, J2 Conn_01x15, J3 DEBUG, J4 QwST, U1 878-APS6404L-3SQR-SN, U2 878-APS6404L-3SQR-SN

Commit message: Moving towards v1
Parts:
- J4: footprint Connector_JST:JST_SH_SM04B-SRSS-TB_1x04-1MP_P1.00mm_Horizontal -> Connector_JST:JST_SH_BM04B-SRSS-TB_1x04-1MP_P1.00mm_Vertical; JLC C160404 -> C160390
Changed lines of the file:
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@@
 			)
 		)
-		(property "Footprint" "Connector_JST:JST_SH_SM04B-SRSS-TB_1x04-1MP_P1.00mm_Horizontal"
+		(property "Footprint" "Connector_JST:JST_SH_BM04B-SRSS-TB_1x04-1MP_P1.00mm_Vertical"
 			(at 160.02 50.8 0)
 			(effects
@@
 			)
 		)
-		(property "JLC" "C160404"
+		(property "JLC" "C160390"
 			(at 160.02 50.8 0)
 			(effects
